Commit message: feat(link_tuner): 参数表画进 2D 图纸、新增一键启动/后端服务
- html: 隐藏 DOM 参数表，改为画进图纸右侧参数栏；躯干宽度联动骨盆半宽
- 新增 pikachu_link_tuner.py 一键启动脚本 + server.py 本地静态/保存服务
- 新增 14dof 连杆调校导出(urdf/xacro/links.json/2d)与 default 默认参数
- xacro: 躯干盒宽度绑定 pelvis_half_width*2 随骨盆联动

Co-Authored-By: Claude <noreply@anthropic.com>

File: urdf/robot/Pikachu_links/default/pikachu_sample_14dof_links.xacro (robot description, xacro)
@@ -6,4 +6,6 @@
   · 每个连杆用 <box> 表示，尺寸/偏移全部参数化，改顶部参数即可整体适配骨骼
   · 单位：米 (m)
+  · 本文件为 14dof 版：手臂只保留 pitch → roll 两段，去掉 yaw 与 elbow
+    （即 19dof 完整版去掉 arm_yaw / elbow 两对关节/连杆）
   与原始 URDF 的对应总表：
     base_link           → 躯干
@@ -13,11 +15,10 @@
     left/right_knee     →ankle      原点沿 -z 偏移 shank_length   （小腿）
     left/right_arm_pitch→roll       可动(revolute)，沿 y 偏移 arm_pitch_to_roll_y
-    left/right_arm_roll →yaw        可动(revolute)，沿 -z 偏移 arm_upper_z
-    left/right_arm_yaw  →elbow      可动(revolute)，沿 -z 偏移 arm_lower_z
+    left/right_arm_roll             下臂末端（14dof 版去掉 yaw/elbow）
     base_link → head_link           可动(revolute)，立于躯干顶 shoulder_height 之上
-    注：臂 pitch/roll/yaw/elbow 与 head 原本为 fixed，这里改成 revolute 以便驱动；
+    注：臂 pitch/roll 与 head 原本为 fixed，这里改成 revolute 以便驱动；
         限位由 arm_lim_* / head_lim_* 控制。
 ============================================================================ -->
-<robot name="pikachu_sample_links" xmlns:xacro="http://www.ros.org/wiki/xacro">
+<robot name="pikachu_sample_14dof_links" xmlns:xacro="http://www.ros.org/wiki/xacro">
   <!-- ============================================================ -->
   <!-- 【集中参数区】改这里即可整体调整 / 适配骨骼模型              -->
@@ -55,7 +56,5 @@
     <!-- 臂 pitch→roll 沿 y 偏移 -->
   <xacro:property name="arm_upper_z" value="0.051"/>
-    <!-- 臂 roll 段：沿 -z 偏移 / 长度 -->
-  <xacro:property name="arm_lower_z" value="0.021"/>
-    <!-- 臂 yaw 段：沿 -z 偏移 / 长度 -->
+    <!-- 臂 roll 段：沿 -z 偏移 / 长度（14dof 版为末端，已去掉 yaw/elbow） -->
   <xacro:property name="arm_thick_x" value="0.03"/>
   <xacro:property name="arm_width_y" value="0.03"/>
@@ -71,7 +70,7 @@
   <!-- ==== 手臂 / 头 关节限位（把 fixed 改成 revolute 后可驱动） ==== -->
   <xacro:property name="arm_lim_min" value="-1.57"/>
-    <!-- 臂 pitch/roll/yaw/elbow 的关节下限（弧度） -->
+    <!-- 臂 pitch/roll 的关节下限（弧度） -->
   <xacro:property name="arm_lim_max" value="1.57"/>
-    <!-- 臂 pitch/roll/yaw/elbow 的关节上限（弧度） -->
+    <!-- 臂 pitch/roll 的关节上限（弧度） -->
   <xacro:property name="head_lim_min" value="-0.8"/>
     <!-- 头关节下限（弧度） -->
@@ -96,9 +95,5 @@
     <!-- 臂段A(arm_pitch 肩)：紫 -->
   <xacro:property name="mat_arm_roll"      value="1.00 0.90 0.25 1"/>
-    <!-- 臂段B(arm_roll 上臂)：黄 -->
-  <xacro:property name="mat_arm_yaw"       value="0.30 0.85 0.80 1"/>
-    <!-- 臂段C(arm_yaw 下臂)：青 -->
-  <xacro:property name="mat_arm_elbow"     value="1.00 0.45 0.55 1"/>
-    <!-- 臂段D(elbow 手)：珊瑚 -->
+    <!-- 臂段B(arm_roll 上臂，14dof 末端)：黄 -->
   <!-- ============================================================ -->
   <!-- 材质定义（每段独立颜色，左右对称共用同一套）              -->
@@ -130,10 +125,4 @@
   <material name="arm_roll">
     <color rgba="${mat_arm_roll}"/>
-  </material>
-  <material name="arm_yaw">
-    <color rgba="${mat_arm_yaw}"/>
-  </material>
-  <material name="arm_elbow">
-    <color rgba="${mat_arm_elbow}"/>
   </material>
   <!-- ============================================================ -->
@@ -222,5 +211,5 @@
   </xacro:macro>
   <!-- ============================================================ -->
-  <!-- 手臂宏：生成 pitch/roll/yaw/elbow 四个 link（全部 revolute 可动） -->
+  <!-- 手臂宏：只生成 pitch → roll 两个 link（14dof，全部 revolute 可动） -->
   <!-- ============================================================ -->
   <xacro:macro name="arm_links" params="side sn">
@@ -242,5 +231,5 @@
       <limit lower="${arm_lim_min}" upper="${arm_lim_max}" effort="2.0" velocity="2"/>
     </joint>
-    <!-- arm_roll_link：上臂段（arm_upper_z） -->
+    <!-- arm_roll_link：下臂/末端段（arm_upper_z）——14dof 版已去掉 yaw/elbow -->
     <link name="${side}_arm_roll_link">
       <visual>
@@ -250,38 +239,4 @@
         </geometry>
         <material name="arm_roll"/>
-      </visual>
-    </link>
-    <joint name="${side}_arm_yaw_joint" type="revolute">
-      <origin xyz="0 0 ${-arm_upper_z}" rpy="0 0 0"/>
-      <parent link="${side}_arm_roll_link"/>
-      <child  link="${side}_arm_yaw_link"/>
-      <axis xyz="0 0 ${sn}"/>
-      <limit lower="${arm_lim_min}" upper="${arm_lim_max}" effort="2.0" velocity="2"/>
-    </joint>
-    <!-- arm_yaw_link：下臂段（arm_lower_z） -->
-    <link name="${side}_arm_yaw_link">
-      <visual>
-        <origin xyz="0 0 ${-arm_lower_z/2.0}" rpy="0 0 0"/>
-        <geometry>
-          <box size="${arm_thick_x} ${arm_width_y} ${arm_lower_z}"/>
-        </geometry>
-        <material name="arm_yaw"/>
-      </visual>
-    </link>
-    <joint name="${side}_elbow_joint" type="revolute">
-      <origin xyz="0 0 ${-arm_lower_z}" rpy="0 -1.57 0"/>
-      <parent link="${side}_arm_yaw_link"/>
-      <child  link="${side}_elbow_link"/>
-      <axis xyz="0 ${-sn} 0"/>
-      <limit lower="${arm_lim_min}" upper="${arm_lim_max}" effort="2.0" velocity="2"/>
-    </joint>
-    <!-- elbow_link：手（末端） -->
-    <link name="${side}_elbow_link">
-      <visual>
-        <origin xyz="0 0 ${-arm_thick_x/2.0}" rpy="0 0 0"/>
-        <geometry>
-          <box size="${arm_thick_x} ${arm_width_y} ${arm_thick_x}"/>
-        </geometry>
-        <material name="arm_elbow"/>
       </visual>
     </link>

File: urdf/robot/Pikachu_links/pikachu_sample_14dof_links_t50_s70_export/pikachu_sample_14dof_links_t50_s70.xacro (robot description, xacro)
@@ -6,4 +6,6 @@
   · 每个连杆用 <box> 表示，尺寸/偏移全部参数化，改顶部参数即可整体适配骨骼
   · 单位：米 (m)
+  · 本文件为 14dof 版：手臂只保留 pitch → roll 两段，去掉 yaw 与 elbow
+    （即 19dof 完整版去掉 arm_yaw / elbow 两对关节/连杆）
   与原始 URDF 的对应总表：
     base_link           → 躯干
@@ -13,20 +15,19 @@
     left/right_knee     →ankle      原点沿 -z 偏移 shank_length   （小腿）
     left/right_arm_pitch→roll       可动(revolute)，沿 y 偏移 arm_pitch_to_roll_y
-    left/right_arm_roll →yaw        可动(revolute)，沿 -z 偏移 arm_upper_z
-    left/right_arm_yaw  →elbow      可动(revolute)，沿 -z 偏移 arm_lower_z
+    left/right_arm_roll             下臂末端（14dof 版去掉 yaw/elbow）
     base_link → head_link           可动(revolute)，立于躯干顶 shoulder_height 之上
-    注：臂 pitch/roll/yaw/elbow 与 head 原本为 fixed，这里改成 revolute 以便驱动；
+    注：臂 pitch/roll 与 head 原本为 fixed，这里改成 revolute 以便驱动；
         限位由 arm_lim_* / head_lim_* 控制。
 ============================================================================ -->
-<robot name="pikachu_sample_links" xmlns:xacro="http://www.ros.org/wiki/xacro">
+<robot name="pikachu_sample_14dof_links" xmlns:xacro="http://www.ros.org/wiki/xacro">
   <!-- ============================================================ -->
   <!-- 【集中参数区】改这里即可整体调整 / 适配骨骼模型              -->
   <!-- ============================================================ -->
   <!-- ==== 躯干 / 肩 ==== -->
-  <xacro:property name="pelvis_half_width" value="0.0515"/>
+  <xacro:property name="pelvis_half_width" value="0.0974"/>
     <!-- 骨盆半宽：躯干中轴线 → 髋 pitch 关节的横向(y)距离，左右腿共用 -->
   <xacro:property name="shoulder_height"   value="0.2"/>
     <!-- 肩高：髋 pitch 平面 → 臂 pitch 关节的 z 抬升（也是躯干盒高度） -->
-  <xacro:property name="torso_len_x"       value="0.08"/>
+  <xacro:property name="torso_len_x"       value="0.1"/>
     <!-- 躯干盒 x(前后) 厚度 -->
   <!-- 躯干盒 y(左右) 宽度已绑定 pelvis_half_width*2：随骨盆联动，
@@ -38,7 +39,7 @@
     <!-- hip_roll→hip_yaw 关节沿 -z 偏移（骨盆下沿） -->
   <!-- ==== 【腿纵向骨长】适配骨骼时重点调这两项 ==== -->
-  <xacro:property name="thigh_length" value="0.025"/>
+  <xacro:property name="thigh_length" value="0.0501"/>
     <!-- 大腿：hip_yaw→knee 关节 沿 -z 偏移（也是该段 box 的长度） -->
-  <xacro:property name="shank_length" value="0.070"/>
+  <xacro:property name="shank_length" value="0.07"/>
     <!-- 小腿：knee→ankle 关节 沿 -z 偏移（也是该段 box 的长度） -->
   <!-- ==== 腿截面尺寸 ==== -->
@@ -52,12 +53,10 @@
   <xacro:property name="foot_hgt_z" value="0.02"/>
   <!-- ==== 臂（fixed，不会动，只做占位） ==== -->
-  <xacro:property name="arm_pitch_to_roll_y" value="0.049"/>
+  <xacro:property name="arm_pitch_to_roll_y" value="0.0682"/>
     <!-- 臂 pitch→roll 沿 y 偏移 -->
-  <xacro:property name="arm_upper_z" value="0.051"/>
-    <!-- 臂 roll 段：沿 -z 偏移 / 长度 -->
-  <xacro:property name="arm_lower_z" value="0.021"/>
-    <!-- 臂 yaw 段：沿 -z 偏移 / 长度 -->
-  <xacro:property name="arm_thick_x" value="0.03"/>
-  <xacro:property name="arm_width_y" value="0.03"/>
+  <xacro:property name="arm_upper_z" value="0.0918"/>
+    <!-- 臂 roll 段：沿 -z 偏移 / 长度（14dof 版为末端，已去掉 yaw/elbow） -->
+  <xacro:property name="arm_thick_x" value="0.0399"/>
+  <xacro:property name="arm_width_y" value="0.0333"/>
   <!-- ==== 头（原始 URDF 没有，适配骨骼时按需调整） ==== -->
   <xacro:property name="head_len_x"         value="0.09"/>
@@ -71,7 +70,7 @@
   <!-- ==== 手臂 / 头 关节限位（把 fixed 改成 revolute 后可驱动） ==== -->
   <xacro:property name="arm_lim_min" value="-1.57"/>
-    <!-- 臂 pitch/roll/yaw/elbow 的关节下限（弧度） -->
+    <!-- 臂 pitch/roll 的关节下限（弧度） -->
   <xacro:property name="arm_lim_max" value="1.57"/>
-    <!-- 臂 pitch/roll/yaw/elbow 的关节上限（弧度） -->
+    <!-- 臂 pitch/roll 的关节上限（弧度） -->
   <xacro:property name="head_lim_min" value="-0.8"/>
     <!-- 头关节下限（弧度） -->
@@ -96,9 +95,5 @@
     <!-- 臂段A(arm_pitch 肩)：紫 -->
   <xacro:property name="mat_arm_roll"      value="1.00 0.90 0.25 1"/>
-    <!-- 臂段B(arm_roll 上臂)：黄 -->
-  <xacro:property name="mat_arm_yaw"       value="0.30 0.85 0.80 1"/>
-    <!-- 臂段C(arm_yaw 下臂)：青 -->
-  <xacro:property name="mat_arm_elbow"     value="1.00 0.45 0.55 1"/>
-    <!-- 臂段D(elbow 手)：珊瑚 -->
+    <!-- 臂段B(arm_roll 上臂，14dof 末端)：黄 -->
   <!-- ============================================================ -->
   <!-- 材质定义（每段独立颜色，左右对称共用同一套）              -->
@@ -130,10 +125,4 @@
   <material name="arm_roll">
     <color rgba="${mat_arm_roll}"/>
-  </material>
-  <material name="arm_yaw">
-    <color rgba="${mat_arm_yaw}"/>
-  </material>
-  <material name="arm_elbow">
-    <color rgba="${mat_arm_elbow}"/>
   </material>
   <!-- ============================================================ -->
@@ -222,5 +211,5 @@
   </xacro:macro>
   <!-- ============================================================ -->
-  <!-- 手臂宏：生成 pitch/roll/yaw/elbow 四个 link（全部 revolute 可动） -->
+  <!-- 手臂宏：只生成 pitch → roll 两个 link（14dof，全部 revolute 可动） -->
   <!-- ============================================================ -->
   <xacro:macro name="arm_links" params="side sn">
@@ -242,5 +231,5 @@
       <limit lower="${arm_lim_min}" upper="${arm_lim_max}" effort="2.0" velocity="2"/>
     </joint>
-    <!-- arm_roll_link：上臂段（arm_upper_z） -->
+    <!-- arm_roll_link：下臂/末端段（arm_upper_z）——14dof 版已去掉 yaw/elbow -->
     <link name="${side}_arm_roll_link">
       <visual>
@@ -250,38 +239,4 @@
         </geometry>
         <material name="arm_roll"/>
-      </visual>
-    </link>
-    <joint name="${side}_arm_yaw_joint" type="revolute">
-      <origin xyz="0 0 ${-arm_upper_z}" rpy="0 0 0"/>
-      <parent link="${side}_arm_roll_link"/>
-      <child  link="${side}_arm_yaw_link"/>
-      <axis xyz="0 0 ${sn}"/>
-      <limit lower="${arm_lim_min}" upper="${arm_lim_max}" effort="2.0" velocity="2"/>
-    </joint>
-    <!-- arm_yaw_link：下臂段（arm_lower_z） -->
-    <link name="${side}_arm_yaw_link">
-      <visual>
-        <origin xyz="0 0 ${-arm_lower_z/2.0}" rpy="0 0 0"/>
-        <geometry>
-          <box size="${arm_thick_x} ${arm_width_y} ${arm_lower_z}"/>
-        </geometry>
-        <material name="arm_yaw"/>
-      </visual>
-    </link>
-    <joint name="${side}_elbow_joint" type="revolute">
-      <origin xyz="0 0 ${-arm_lower_z}" rpy="0 -1.57 0"/>
-      <parent link="${side}_arm_yaw_link"/>
-      <child  link="${side}_elbow_link"/>
-      <axis xyz="0 ${-sn} 0"/>
-      <limit lower="${arm_lim_min}" upper="${arm_lim_max}" effort="2.0" velocity="2"/>
-    </joint>
-    <!-- elbow_link：手（末端） -->
-    <link name="${side}_elbow_link">
-      <visual>
-        <origin xyz="0 0 ${-arm_thick_x/2.0}" rpy="0 0 0"/>
-        <geometry>
-          <box size="${arm_thick_x} ${arm_width_y} ${arm_thick_x}"/>
-        </geometry>
-        <material name="arm_elbow"/>
       </visual>
     </link>
