Commit message: fix(retarget) 21dof 默认 + arm_roll 去 90°对正 + URDF 关节轴方向规范化 + head 三映射
- Pikachu_Retarget: 默认 URDF 从 14dof 切到 21dof
- npz_row_to_urdf 去掉 arm_roll ±90° 硬编码 (本批 npz 的 arm_roll 0 即与
  21dof URDF 装配位对齐, 反推 limit 方向会超限位造成镜像翻折)
- blender_urdf_map: head_joint 单骨拆分/补全 head_yaw/roll/pitch 三映射
- 21dof.urdf: 髋/膝/踝/肩等多关节 axis 取反 + limit 对调 (方向规范化)

Co-Authored-By: Claude Code <noreply@anthropic.com>

File: urdf/robot/Pikachu_V025/urdf/Pikachu_V025_flat_21dof.urdf (robot description, URDF)
Before this commit: robot Pikachu_V025, 22 links, 21 joints
Joints:
- joint left_ankle_joint: axis 0 -1 0 -> 0 1 0; limit lower=-0.52 upper=1.05 effort=9.0 velocity=2 -> lower=-1.05 upper=0.52 effort=9.0 velocity=2
- joint left_arm_pitch_joint: axis 0 -1 0 -> 0 1 0; limit lower=-1.05 upper=3.14 effort=9 velocity=2 -> lower=-3.14 upper=1.05 effort=9 velocity=2
- joint left_elbow_ankle_joint: axis 0 -1 0 -> 0 1 0; limit lower=0 upper=2.44 effort=9 velocity=2 -> lower=-2.44 upper=0 effort=9 velocity=2
- joint left_hip_pitch_joint: axis 0 -1 0 -> 0 1 0; limit lower=0 upper=2.44 effort=12.5 velocity=2 -> lower=-2.44 upper=0 effort=12.5 velocity=2
- joint left_hip_yaw_joint: axis 0 0 1 -> 0 0 -1; limit lower=-0.09 upper=0.26 effort=9.0 velocity=1 -> lower=-0.26 upper=0.09 effort=9.0 velocity=1
- joint left_knee_joint: axis 0 1 0 -> 0 -1 0; limit lower=0 upper=1.57 effort=12.5 velocity=3 -> lower=-1.57 upper=0.09 effort=12.5 velocity=3
- joint right_arm_roll_joint: axis -1 0 0 -> 1 0 0; limit lower=0.0 upper=1.57 effort=9 velocity=2 -> lower=-1.57 upper=0 effort=9 velocity=2
- joint right_hip_roll_joint: axis -1 0 0 -> 1 0 0; limit lower=-0.09 upper=0.26 effort=9.0 velocity=1 -> lower=-0.26 upper=0.09 effort=9.0 velocity=1
